Commit message: ur3_man bringup

File: ur3_man_description/urdf/kinect_v2.urdf.xacro (robot description, xacro)
@@ -21,5 +21,5 @@
     <link name="kinect2_link"/>
     <joint name="${prefix}_joint" type="fixed">
-      <origin xyz="0.02 -0.05 0.045" rpy="${-pi/2+0.1} 0 ${-pi/2}" />
+      <origin xyz="0.01 -0.097 0.045" rpy="${-pi/2+0.1} 0 ${-pi/2}" />
       <parent link="${prefix}_base"/>
       <child link="kinect2_link"/>

File: ur3_man_description/urdf/robotiq_gripper.urdf.xacro (robot description, xacro)
@@ -1,5 +1,4 @@
 <?xml version="1.0"?>
 <robot xmlns:xacro="http://www.ros.org/wiki/xacro" name="robotiq_gripper">
-  <xacro:include filename="$(find robotiq_85_description)/urdf/robotiq_85_gripper.urdf.xacro" />
   <xacro:property name="M_PI" value="3.1415926535897931" />
   <gazebo>

File: ur3_man_description/urdf/ur3_man_robot.urdf.xacro (robot description, xacro)
@@ -73,4 +73,10 @@
     <origin xyz="0.008 0 0" rpy="0 0 0"/>
   </xacro:robotiq_85_gripper>
+  <link name="left_gripper_ee_link"/>
+  <joint name="left_gripper_ee_joint" type="fixed">
+    <origin xyz="0.13 0 0" rpy="0 0 0"/>
+    <parent link="left_gripper_base_link"/>
+    <child link="left_gripper_ee_link"/>
+  </joint>
   <!-- right_gripper -->
   <xacro:robotiq_gripper_coupling parent="right_arm_ee_link" prefix="right_">
@@ -80,3 +86,9 @@
     <origin xyz="0.008 0 0" rpy="0 0 0"/>
   </xacro:robotiq_85_gripper>
+  <link name="right_gripper_ee_link"/>
+  <joint name="right_gripper_ee_joint" type="fixed">
+    <origin xyz="0.13 0 0" rpy="0 0 0"/>
+    <parent link="right_gripper_base_link"/>
+    <child link="right_gripper_ee_link"/>
+  </joint>
 </robot>
